Commit message: fix(sim): 무명령 활주 물리 수정 — 바퀴 dynamics/maxVel/mu 조정 (report §1.22 ✅)
- 활주 중 바퀴가 안 굴러 odom 정지 인식 → AMCL belief 동결 → 실위치와
  1.2m 간극 → 'Starting point in lethal space'로 F1 pickup ABORT 2회 재현
- 수정: 바퀴 조인트 damping 0.05/friction 0.3, 접촉 maxVel 1→0, mu 1→100
- A/B 실측: 30초당 8.6cm → 90초당 2.4mm (~1/100)
- §1.22 '미션 중 무해' 오판 정정 + 완료 처리

Co-Authored-By: Claude Fable 5 <noreply@anthropic.com>

File: src/common_pkg/urdf/delivery_robot.urdf.xacro (robot description, xacro)
@@ -81,4 +81,5 @@
     <origin xyz="0 0.25662 0.013" rpy="0 0 0"/>  <!-- ★SIM z 0.033->0.013 (base 0.02 보정) -->
     <axis xyz="0 1 0"/>
+    <dynamics damping="0.05" friction="0.3"/>  <!-- ★SIM 무명령 활주 제동 (§1.22) — max_wheel_torque 40 대비 미미 -->
   </joint>
   <link name="right_wheel">
@@ -104,4 +105,5 @@
     <origin xyz="0 -0.25662 0.013" rpy="0 0 0"/>  <!-- ★SIM z 0.033->0.013 (base 0.02 보정) -->
     <axis xyz="0 1 0"/>
+    <dynamics damping="0.05" friction="0.3"/>  <!-- ★SIM 무명령 활주 제동 (§1.22) -->
   </joint>
   <!-- ============================================================
@@ -229,15 +231,16 @@
        ============================================================ -->
   <!-- 바퀴 마찰 (없으면 헛바퀴) -->
+  <!-- ★SIM maxVel 0: 접촉 보정속도 주입 차단(무명령 활주 §1.22), mu 100: 슬립 방지 -->
   <gazebo reference="left_wheel">
-    <mu1>1.0</mu1><mu2>1.0</mu2>
+    <mu1>100.0</mu1><mu2>100.0</mu2>
     <kp>1000000.0</kp><kd>100.0</kd>
-    <minDepth>0.001</minDepth><maxVel>1.0</maxVel>
+    <minDepth>0.001</minDepth><maxVel>0.0</maxVel>
     <fdir1>1 0 0</fdir1>
     <material>Gazebo/Black</material>
   </gazebo>
   <gazebo reference="right_wheel">
-    <mu1>1.0</mu1><mu2>1.0</mu2>
+    <mu1>100.0</mu1><mu2>100.0</mu2>
     <kp>1000000.0</kp><kd>100.0</kd>
-    <minDepth>0.001</minDepth><maxVel>1.0</maxVel>
+    <minDepth>0.001</minDepth><maxVel>0.0</maxVel>
     <fdir1>1 0 0</fdir1>
     <material>Gazebo/Black</material>
@@ -247,5 +250,5 @@
     <mu1>0.0</mu1><mu2>0.0</mu2>
     <kp>1000000.0</kp><kd>100.0</kd>
-    <minDepth>0.001</minDepth><maxVel>1.0</maxVel>
+    <minDepth>0.001</minDepth><maxVel>0.0</maxVel>
     <material>Gazebo/Black</material>
   </gazebo>
@@ -253,5 +256,5 @@
     <mu1>0.0</mu1><mu2>0.0</mu2>
     <kp>1000000.0</kp><kd>100.0</kd>
-    <minDepth>0.001</minDepth><maxVel>1.0</maxVel>
+    <minDepth>0.001</minDepth><maxVel>0.0</maxVel>
     <material>Gazebo/Black</material>
   </gazebo>

Commit message: fix(sim): 적대 리뷰 P0/P1 반영 — 바퀴 fdir1 차축+캐스터 마찰(크리프 근절), 보행자 init 복원·참값 근접, 스모크 핫픽스 12건, 정적 장애물·리프트 mock, 행위 테스트 추가
- URDF: fdir1 0 0 1(차축, collision 프레임) + 캐스터 mu 0.5 — check_idle_drift 0.5425m→0.0000m/90s,
  주행 후 정지 활주 0, θ90 퇴화 자발 회전 제거 (표준 ODE 하네스+스택 검증, §1.26)
- pedestrians.py: __init__ 복원(a6a5115 회귀), 근접 판정 /gazebo/model_states 참값 우선
- smoke: INT/TERM trap rc, RUN_DIR 계약, request_switch success=True 판정+armed 앵커, cancel_goal 후 재시도,
  finalize 멱등·trap 호출, missed-rate fail-closed·finalize 이전, profiler flush, wait_for_* timeout,
  realign 수치 검증, 팔 완료 층별 쌍, 실패 attempt 로그 보존, SKIP_BUILD, gzserver 종료 대기
- repeat: RUN_DIR 파싱, retries/realign 열, cgroup v1/v2 OOM 가드, MAX_MISSED_RATE=30, SKIP_BUILD 2회차~
- 정적 장애물(경로 위, static=true, 레인 간격 테스트), 리프트 mock(joint_pose_trajectory+자기잠금 friction, frame_id world)
- contract 테스트 확장(AST 가드·핫픽스·물리 고정) + test_pedestrians_stub/test_static_obstacles_layout (오프라인 28/28)
- improvement_report §1.26 ✅ / §1.27 [70%]

Co-Authored-By: Claude Fable 5 <noreply@anthropic.com>

File: src/common_pkg/urdf/delivery_robot.urdf.xacro (robot description, xacro)
@@ -226,4 +226,10 @@
     <axis xyz="0 0 1"/>
     <limit lower="0.0" upper="0.5" effort="50" velocity="0.05"/>
+    <!-- ★SIM 자기잠금(웜기어+T스크류 등가): joint_pose_trajectory 플러그인은 마지막
+         포인트 적용 후 조인트를 놓는다(has_trajectory=false) — 마찰 없이는 캐리어가
+         중력으로 낙하해 리프트 "상승 유지" 검증이 플래키해진다(2026-08-20). ODE 조인트
+         friction 은 vel=0 모터(FMax=friction)로 구현되어 위치를 유지한다. 실기 하중
+         5kg·캐리어 0.5kg 기준 20N 이면 충분(effort 50 이내). -->
+    <dynamics damping="1.0" friction="20.0"/>
   </joint>
   <!-- ============================================================
@@ -231,27 +237,41 @@
        ============================================================ -->
   <!-- 바퀴 마찰 (없으면 헛바퀴) -->
-  <!-- ★SIM maxVel 0: 접촉 보정속도 주입 차단(무명령 활주 §1.22).
-       mu1 100 / mu2 1.0 방향 분리(2026-08-18, §1.25g): 활주는 구름 방향(mu1)이
-       지배해 100 유지 — mu 30 균일로 낮추자 활주 0.55m/90s 재발 실측.
-       전복은 횡방향 그립(mu2)이 지배 — 벽 접촉 회복기동에서 mu 100 그립 토크가
-       로봇을 90° 옆으로 뒤집는 사례 2회 실측(분산 run2). mu2=1.0 은 횡력 상한을
-       체중 1배로 캡해 전복 임계(~1.8배) 미달 → 물리적으로 side-flip 불가. -->
+  <!-- ★SIM maxVel 0: 접촉 보정속도 주입 차단(§1.22). mu 100/100: 슬립 방지.
+       fdir1="0 0 1" = 차축 방향 (2026-08-20/21 확정, docs/session_wiki/2026-08-20_review_followup):
+       Gazebo 11 은 fdir1 을 collision WorldPose 로 회전한다(소스 확인). 바퀴 collision 은
+       rpy 1.5708 로 눕혀져 collision z = 링크 -y = 차축 → 바퀴가 굴러도 불변.
+       구 "1 0 0"(구름 방향)은 바퀴와 함께 회전해 θ≈90° 마다 마찰축이 접지 법선과 겹치는
+       퇴화 창을 만든다 — 표준 ODE 하네스(바퀴각 0/45/80/90° 프리셋, 0.03g 횡 밀기)에서
+       θ90 yaw 1.6 rad 자발 회전, 스택 stop_probe 에서는 주행 후 정지 30s 에 −0.63m 이동
+       + 이후 전진 명령에 후진(뒤집힌 yaw) 재현. "0 1 0"(collision y = 링크 z) 은 θ0 에서
+       퇴화. 차축 fdir1 은 전 각도·전 방향 안정(하네스 1/2 전수 0 이동).
+       (구 mu2=1.0 "횡력 캡 → 전복 1.8배 미달" 논리는 폐기: 1.8 은 마스트+LiDAR 누락
+       산술 오류로 실제 1.465g 이고, 전복·정지 중 회전의 구동원은 fdir1 퇴화였다.)
+       ※ 차축 fdir1 + 무마찰 캐스터(mu 0) 조합은 ODE 가 6mm/s 등속 전진 크리프를 만든다
+       (기동 직후·정지 후 모두, 결정적) — 원인 분리: 플러그인/ROS/월드/스폰 무관, 순수
+       gzserver 재현, 캐스터 마찰만이 차이. 해법은 캐스터 마찰(아래). 마찰/스프링 값
+       변경 시 check_idle_drift.sh 재실측 필수. -->
   <gazebo reference="left_wheel">
-    <mu1>100.0</mu1><mu2>1.0</mu2>
+    <mu1>100.0</mu1><mu2>100.0</mu2>
     <kp>1000000.0</kp><kd>100.0</kd>
     <minDepth>0.001</minDepth><maxVel>0.0</maxVel>
-    <fdir1>1 0 0</fdir1>
+    <fdir1>0 0 1</fdir1>
     <material>Gazebo/Black</material>
   </gazebo>
   <gazebo reference="right_wheel">
-    <mu1>100.0</mu1><mu2>1.0</mu2>
+    <mu1>100.0</mu1><mu2>100.0</mu2>
     <kp>1000000.0</kp><kd>100.0</kd>
     <minDepth>0.001</minDepth><maxVel>0.0</maxVel>
-    <fdir1>1 0 0</fdir1>
+    <fdir1>0 0 1</fdir1>
     <material>Gazebo/Black</material>
   </gazebo>
-  <!-- 볼 캐스터(앞/뒤): 마찰 0 으로 자유 미끄럼 -->
+  <!-- 볼 캐스터(앞/뒤): 고정 구 + 마찰 0.5 (2026-08-21). 구 설정 mu 0(무마찰 자유 미끄럼)은
+       차축 fdir1 바퀴와 조합될 때 ODE 가 6mm/s 등속 크리프를 만들었다(정지 중 odom 불변 활주
+       → AMCL belief 드리프트 0.7~1.0m 의 근원, §1.22/§1.25h). 순수 gzserver 스윕: 캐스터
+       mu 0 → 6.1mm/s, 0.05 → 5.0mm/s, 0.3/1.0/3.0 → 0. 0.5 는 여유를 둔 값 — 스키드 드래그
+       0.5×캐스터 하중(~25N) ≈ 12N 로 구동 여유(바퀴당 40N·m/0.033m) 대비 ~1%, 정지 시
+       파킹 브레이크 역할. 실물 볼 캐스터는 구름(구름저항 1~3%)이므로 시뮬 전용 근사값. -->
   <gazebo reference="caster_wheel">
-    <mu1>0.0</mu1><mu2>0.0</mu2>
+    <mu1>0.5</mu1><mu2>0.5</mu2>
     <kp>1000000.0</kp><kd>100.0</kd>
     <minDepth>0.001</minDepth><maxVel>0.0</maxVel>
@@ -259,5 +279,5 @@
   </gazebo>
   <gazebo reference="caster_wheel_front">
-    <mu1>0.0</mu1><mu2>0.0</mu2>
+    <mu1>0.5</mu1><mu2>0.5</mu2>
     <kp>1000000.0</kp><kd>100.0</kd>
     <minDepth>0.001</minDepth><maxVel>0.0</maxVel>
@@ -299,4 +319,17 @@
     </plugin>
   </gazebo>
+  <!-- ★SIM 리프트 구동 (2026-08-20): lift_joint 를 시뮬에서 움직일 수단.
+       /set_lift_trajectory (trajectory_msgs/JointTrajectory) 수신 시 조인트를
+       목표 위치로 보간 이동. 실기는 웜기어+T스크류 컨트롤러가 담당(§hardware_spec)
+       — 이 플러그인은 시뮬 mock. 사용처: smoke 의 lift_cycle.py (WITH_LIFT=1). -->
+  <gazebo>
+    <plugin name="lift_trajectory" filename="libgazebo_ros_joint_pose_trajectory.so">
+      <ros>
+        <namespace>/</namespace>
+        <remapping>set_joint_trajectory:=set_lift_trajectory</remapping>
+      </ros>
+      <update_rate>10</update_rate>
+    </plugin>
+  </gazebo>
   <!-- LiDAR 센서 (RPLiDAR A1 근사: 360도, 8m), frame_name=laser -->
   <gazebo reference="laser">

Commit message: sync(jetson): 젯슨 Code_Space 작업 트리 반영 — 2026-09-12 10:31:54 KST
직전 반영 대비 변경:
M	README.md
M	TODO.md
A	docker/compose/docker-compose.jetson.mapping.yml
M	docs/deployment/01_portability_policy.md
M	docs/deployment/02_opencr_serial_protocol.md
A	docs/deployment/04_field_mapping_navigation.md
A	scripts/arm_node_safe_probe.py
M	scripts/build_handheld_mapping.sh
M	scripts/check_handheld_mapping.sh
M	scripts/dds_contract_probe.py
M	scripts/generate_kku_maps.py
M	scripts/generate_kku_worlds.py
M	scripts/jetson_preflight.py
A	scripts/jetson_thermal_watchdog.sh
M	scripts/log_session.py
A	scripts/nav_safety_gate_probe.py
M	scripts/probe_rplidar_node.sh
M	scripts/run_arm_press.py
M	scripts/run_field_mapping.sh
M	scripts/run_offline_tests.sh
A	scripts/save_field_map.sh
M	scripts/save_handheld_map.sh
A	scripts/start_field_base.sh
A	scripts/start_field_mapping.sh
A	scripts/start_field_navigation.sh
M	scripts/start_handheld_mapping.sh
M	scripts/stop_handheld_mapping.sh
M	scripts/sync_docs_to_notion.py
A	scripts/synthetic_stationary_base.py
M	scripts/test_arm_execution_contract.py
A	scripts/test_arm_node_safe_runtime.sh
M	scripts/test_arm_sequence.py
M	scripts/test_diff_drive_odometry.py
M	scripts/test_field_mapping_launch.py
M	scripts/test_field_scripts_contract.py
A	scripts/test_field_transition_save.sh
M	scripts/test_jetson_dds_contract.sh
M	scripts/test_jetson_image_runtime.py
M	scripts/test_jetson_safe_profiles.py
M	scripts/test_kku_navigation_launch.py
A	scripts/test_map_contract.py
A	scripts/test_nav_safety_gate.py
A	scripts/test_nav_safety_gate_runtime.sh
M	scripts/test_opencr_bridge_dryrun.py
A	scripts/test_opencr_firmware_contract.py
M	scripts/test_opencr_protocol.py
M	scripts/test_opencr_safety_contract.py
M	scripts/test_udev_contract.py
M	scripts/verify_jetson_source_in_container.sh
M	src/common_pkg/urdf/delivery_robot.urdf.xacro
M	src/drive_pkg/CMakeLists.txt
M	src/drive_pkg/config/drive_calib.yaml
A	src/drive_pkg/config/nav_safety.yaml
M	src/drive_pkg/drive_pkg/keyboard_teleop.py
A	src/drive_pkg/drive_pkg/nav_safety_gate.py
M	src/drive_pkg/drive_pkg/opencr_bridge_node.py
M	src/drive_pkg/drive_pkg/opencr_protocol.py
A	src/drive_pkg/drive_pkg/safety_gate.py
A	src/drive_pkg/firmware/opencr/opencr_drive_bridge.ino
M	src/drive_pkg/launch/drive_bringup.launch.py
M	src/slam_pkg/CMakeLists.txt
M	src/slam_pkg/config/nav2_params.yaml
A	src/slam_pkg/launch/field_base.launch.py
A	src/slam_pkg/launch/field_mapping_only.launch.py
M	src/slam_pkg/launch/kku_navigation.launch.py
M	src/slam_pkg/package.xml
A	src/slam_pkg/slam_pkg/__init__.py
A	src/slam_pkg/slam_pkg/map_contract.py
A	watchdog_logs/20260911-232300_JETSON_WATCHDOG/monitor_anomalies.log
A	watchdog_logs/20260911-232300_JETSON_WATCHDOG/thermal_watchdog.log

젯슨 HEAD c83d092cc (lee/hw-design-review) 에 미커밋 변경 92개(수정 39 · 추가 53 · 삭제 0)를 얹은 스냅샷이다.
읽기 전용(git-upload-pack · ls-files/hash-object · tar)으로 수집했고 .gitignore 대상, *.bak*, 지도 직렬화 바이너리(maps/**/*.posegraph·*.data)는 뺐다.
모든 blob id 가 젯슨 git hash-object 결과와 일치한다.

Co-Authored-By: Claude Opus 5 <noreply@anthropic.com>

File: src/common_pkg/urdf/delivery_robot.urdf.xacro (robot description, xacro)
@@ -18,4 +18,11 @@
 -->
 <robot name="delivery_robot" xmlns:xacro="http://www.ros.org/wiki/xacro">
+  <!-- 현장 장착값 오버라이드. 기본값은 2026-09-10 모델이며 실측 전 ⚠️미확인. -->
+  <xacro:arg name="laser_x" default="-0.1015"/>
+  <xacro:arg name="laser_y" default="0.0"/>
+  <xacro:arg name="laser_z" default="0.750"/>
+  <xacro:arg name="laser_roll" default="0.0"/>
+  <xacro:arg name="laser_pitch" default="0.0"/>
+  <xacro:arg name="laser_yaw" default="0.0"/>
   <!-- ===== 공통 재질(색상) ===== -->
   <material name="grey">  <color rgba="0.7 0.7 0.7 1.0"/></material>
@@ -175,5 +182,6 @@
     <parent link="base_link"/>
     <child  link="laser"/>
-    <origin xyz="-0.1015 0 0.750" rpy="0 0 0"/>
+    <origin xyz="$(arg laser_x) $(arg laser_y) $(arg laser_z)"
+            rpy="$(arg laser_roll) $(arg laser_pitch) $(arg laser_yaw)"/>
   </joint>
   <!-- ============================================================

Commit message: sync(jetson): 젯슨 Code_Space 작업 트리 반영 — 2026-09-13 20:10:12 KST
직전 반영 대비 변경:
M	scripts/start_field_base.sh
M	src/common_pkg/urdf/delivery_robot.urdf.xacro
M	src/drive_pkg/config/drive_calib.yaml
M	src/slam_pkg/config/nav2_params.yaml
M	src/slam_pkg/launch/field_base.launch.py

젯슨 HEAD c83d092cc (lee/hw-design-review) 에 미커밋 변경 142개(수정 42 · 추가 100 · 삭제 0)를 얹은 스냅샷이다.
읽기 전용(git-upload-pack · ls-files/hash-object · tar)으로 수집했고 .gitignore 대상, 백업 사본(*.bak*·*.orig·*.rej·*.before-*), 지도 직렬화 바이너리(maps/**/*.posegraph·*.data)는 뺐다.
모든 blob id 가 젯슨 git hash-object 결과와 일치한다.

Co-Authored-By: Claude Opus 5 <noreply@anthropic.com>

File: src/common_pkg/urdf/delivery_robot.urdf.xacro (robot description, xacro)
@@ -12,5 +12,5 @@
       (SLAM/Nav2 가 /scan frame_id 를 "laser" 로 기대하므로 정렬)
    3. 바퀴/캐스터 마찰(mu/kp/kd) gazebo 블록
-   4. diff_drive 플러그인 (wheel_separation=0.51324, wheel_diameter=0.066)
+   4. diff_drive 플러그인 (wheel_separation=0.4194, wheel_diameter=0.066)
    5. joint_state_publisher 플러그인 (좌우 바퀴 + lift_joint)
    6. LiDAR ray 센서 플러그인 (360도, 8m, frame_name=laser)
@@ -18,8 +18,8 @@
 -->
 <robot name="delivery_robot" xmlns:xacro="http://www.ros.org/wiki/xacro">
-  <!-- 현장 장착값 오버라이드. 기본값은 2026-09-10 모델이며 실측 전 ⚠️미확인. -->
-  <xacro:arg name="laser_x" default="-0.1015"/>
+  <!-- 현장 장착값 오버라이드. 기본값은 HW팀 r1.urdf v2(2026-09-13) 기준. -->
+  <xacro:arg name="laser_x" default="-0.117"/>
   <xacro:arg name="laser_y" default="0.0"/>
-  <xacro:arg name="laser_z" default="0.750"/>
+  <xacro:arg name="laser_z" default="0.667"/>
   <xacro:arg name="laser_roll" default="0.0"/>
   <xacro:arg name="laser_pitch" default="0.0"/>
@@ -40,5 +40,5 @@
          바퀴 접지면과 같은 평면 -> 섀시가 바닥에 깔려 바퀴 헛돎.
          본체를 0.02 들어올리고 아래에서 바퀴/캐스터를 같은 양 내려 접지 유지. -->
-    <origin xyz="0 0 0.02" rpy="0 0 0"/>
+    <origin xyz="0 0 0" rpy="0 0 0"/>  <!-- r1 v2: 섀시 바닥 z=0.053 이라 들어올림 보정 불필요 -->
   </joint>
   <!-- ============================================================
@@ -47,32 +47,32 @@
   <link name="base_link">
     <visual>
-      <origin xyz="-0.025 0 0.125" rpy="0 0 0"/>
-      <geometry><box size="0.300 0.400 0.250"/></geometry>
+      <origin xyz="-0.147 0 0.178" rpy="0 0 0"/>
+      <geometry><box size="0.360 0.400 0.250"/></geometry>
       <material name="grey"/>
     </visual>
     <collision>
-      <origin xyz="-0.025 0 0.125" rpy="0 0 0"/>
-      <geometry><box size="0.300 0.400 0.250"/></geometry>
-    </collision>
-    <inertial>
-      <origin xyz="-0.025 0 0.125" rpy="0 0 0"/>
+      <origin xyz="-0.147 0 0.178" rpy="0 0 0"/>
+      <geometry><box size="0.360 0.400 0.250"/></geometry>
+    </collision>
+    <inertial>
+      <origin xyz="-0.147 0 0.178" rpy="0 0 0"/>
       <mass value="8.0"/>
       <inertia ixx="0.1483" ixy="0" ixz="0"
-                            iyy="0.1017" iyz="0"
-                                         izz="0.1667"/>
-    </inertial>
-  </link>
-  <!-- ============================================================
-       구동 바퀴 (지름 66 -> 반지름 0.033), 트랙폭 0.51324
+                            iyy="0.1281" iyz="0"
+                                         izz="0.1931"/>
+    </inertial>
+  </link>
+  <!-- ============================================================
+       구동 바퀴 (지름 66 -> 반지름 0.033), 트랙폭 0.4194 (r1 v2)
        ============================================================ -->
   <link name="left_wheel">
     <visual>
       <origin xyz="0 0 0" rpy="1.5708 0 0"/>
-      <geometry><cylinder radius="0.033" length="0.025"/></geometry>
+      <geometry><cylinder radius="0.033" length="0.0178"/></geometry>
       <material name="black"/>
     </visual>
     <collision>
       <origin xyz="0 0 0" rpy="1.5708 0 0"/>
-      <geometry><cylinder radius="0.033" length="0.025"/></geometry>
+      <geometry><cylinder radius="0.033" length="0.0178"/></geometry>
     </collision>
     <inertial>
@@ -86,5 +86,5 @@
     <parent link="base_link"/>
     <child  link="left_wheel"/>
-    <origin xyz="0 0.25662 0.013" rpy="0 0 0"/>  <!-- ★SIM z 0.033->0.013 (base 0.02 보정) -->
+    <origin xyz="0 0.2097 0.033" rpy="0 0 0"/>  <!-- r1 v2 -->
     <axis xyz="0 1 0"/>
     <dynamics damping="0.05" friction="0.3"/>  <!-- ★SIM 무명령 활주 제동 (§1.22) — max_wheel_torque 40 대비 미미 -->
@@ -93,10 +93,10 @@
     <visual>
       <origin xyz="0 0 0" rpy="1.5708 0 0"/>
-      <geometry><cylinder radius="0.033" length="0.025"/></geometry>
+      <geometry><cylinder radius="0.033" length="0.0178"/></geometry>
       <material name="black"/>
     </visual>
     <collision>
       <origin xyz="0 0 0" rpy="1.5708 0 0"/>
-      <geometry><cylinder radius="0.033" length="0.025"/></geometry>
+      <geometry><cylinder radius="0.033" length="0.0178"/></geometry>
     </collision>
     <inertial>
@@ -110,5 +110,5 @@
     <parent link="base_link"/>
     <child  link="right_wheel"/>
-    <origin xyz="0 -0.25662 0.013" rpy="0 0 0"/>  <!-- ★SIM z 0.033->0.013 (base 0.02 보정) -->
+    <origin xyz="0 -0.2097 0.033" rpy="0 0 0"/>  <!-- r1 v2 -->
     <axis xyz="0 1 0"/>
     <dynamics damping="0.05" friction="0.3"/>  <!-- ★SIM 무명령 활주 제동 (§1.22) -->
@@ -120,10 +120,10 @@
     <visual>
       <origin xyz="0 0 0" rpy="0 0 0"/>
-      <geometry><sphere radius="0.015"/></geometry>
+      <geometry><sphere radius="0.033"/></geometry>
       <material name="black"/>
     </visual>
     <collision>
       <origin xyz="0 0 0" rpy="0 0 0"/>
-      <geometry><sphere radius="0.015"/></geometry>
+      <geometry><sphere radius="0.033"/></geometry>
     </collision>
     <inertial>
@@ -135,5 +135,5 @@
     <parent link="base_link"/>
     <child  link="caster_wheel"/>
-    <origin xyz="-0.1285 0 -0.005" rpy="0 0 0"/>  <!-- ★SIM z 0.015->-0.005 (base 0.02 보정) -->
+    <origin xyz="-0.2575 0 0.033" rpy="0 0 0"/>  <!-- r1 v2 -->
   </joint>
   <!-- ★SIM 전방 캐스터 추가. 원본은 후방 캐스터 1개뿐이고 마스트가 앞에 있어
@@ -158,5 +158,5 @@
     <parent link="base_link"/>
     <child  link="caster_wheel_front"/>
-    <origin xyz="0.1285 0 -0.005" rpy="0 0 0"/>
+    <origin xyz="0.1285 0 0.015" rpy="0 0 0"/>  <!-- ★SIM base z=0 에 맞춰 접지 유지 -->
   </joint>
   <!-- ============================================================
@@ -306,5 +306,5 @@
       <left_joint>left_wheel_joint</left_joint>
       <right_joint>right_wheel_joint</right_joint>
-      <wheel_separation>0.51324</wheel_separation>
+      <wheel_separation>0.4194</wheel_separation>
       <wheel_diameter>0.066</wheel_diameter>
       <max_wheel_torque>40.0</max_wheel_torque>          <!-- ★SIM 0.5m/s 가속 여유 -->
